Commit message: joint limit resolved

File: kinova-ros/kinova_description/urdf/j2n6s300.xacro (robot description, xacro)
@@ -57,6 +57,8 @@
     <xacro:property name="joint_2_origin_xyz" value="0 0.0016 -0.11875" />
     <xacro:property name="joint_2_origin_rpy" value="-${J_PI/2} 0 ${J_PI}" />
-    <xacro:property name="joint_2_lower_limit" value="${47/180*J_PI}" />
-    <xacro:property name="joint_2_upper_limit" value="${313/180*J_PI}" />
+    <xacro:property name="joint_2_lower_limit" value="${-2*J_PI}" />
+    <!--<xacro:property name="joint_2_lower_limit" value="${47/180*J_PI}" /> -->
+    <!--<xacro:property name="joint_2_upper_limit" value="${313/180*J_PI}" />-->
+    <xacro:property name="joint_2_upper_limit" value="${2*J_PI}" />-
     <xacro:property name="joint_2_velocity_limit" value="${36*J_PI/180}" />
     <xacro:property name="joint_2_torque_limit" value="80" />
@@ -66,6 +68,8 @@
     <xacro:property name="joint_3_origin_xyz" value="0 -0.410 0" />
     <xacro:property name="joint_3_origin_rpy" value="0 ${J_PI} 0" />
-    <xacro:property name="joint_3_lower_limit" value="${19/180*J_PI}" />
-    <xacro:property name="joint_3_upper_limit" value="${341/180*J_PI}" />
+    <!--<xacro:property name="joint_3_lower_limit" value="${19/180*J_PI}" />
+    <xacro:property name="joint_3_upper_limit" value="${341/180*J_PI}" />-->
+    <xacro:property name="joint_3_lower_limit" value="${-2*J_PI}" />
+    <xacro:property name="joint_3_upper_limit" value="${2*J_PI}" />
     <xacro:property name="joint_3_velocity_limit" value="${36*J_PI/180}" />
     <xacro:property name="joint_3_torque_limit" value="40" />

Commit message: joint limit resolved

File: kinova-ros/kinova_description/urdf/j2n6s300.xacro (robot description, xacro)
@@ -57,8 +57,8 @@
     <xacro:property name="joint_2_origin_xyz" value="0 0.0016 -0.11875" />
     <xacro:property name="joint_2_origin_rpy" value="-${J_PI/2} 0 ${J_PI}" />
-    <xacro:property name="joint_2_lower_limit" value="${-2*J_PI}" />
-    <!--<xacro:property name="joint_2_lower_limit" value="${47/180*J_PI}" /> -->
-    <!--<xacro:property name="joint_2_upper_limit" value="${313/180*J_PI}" />-->
-    <xacro:property name="joint_2_upper_limit" value="${2*J_PI}" />-
+    <xacro:property name="joint_2_lower_limit" value="${47/180*J_PI}" />
+    <xacro:property name="joint_2_upper_limit" value="${313/180*J_PI}" />
+    <!--<xacro:property name="joint_2_lower_limit" value="${-4*J_PI}" />
+    <xacro:property name="joint_2_upper_limit" value="${4*J_PI}" />-->
     <xacro:property name="joint_2_velocity_limit" value="${36*J_PI/180}" />
     <xacro:property name="joint_2_torque_limit" value="80" />
@@ -68,8 +68,8 @@
     <xacro:property name="joint_3_origin_xyz" value="0 -0.410 0" />
     <xacro:property name="joint_3_origin_rpy" value="0 ${J_PI} 0" />
-    <!--<xacro:property name="joint_3_lower_limit" value="${19/180*J_PI}" />
-    <xacro:property name="joint_3_upper_limit" value="${341/180*J_PI}" />-->
-    <xacro:property name="joint_3_lower_limit" value="${-2*J_PI}" />
-    <xacro:property name="joint_3_upper_limit" value="${2*J_PI}" />
+    <xacro:property name="joint_3_lower_limit" value="${19/180*J_PI}" />
+    <xacro:property name="joint_3_upper_limit" value="${341/180*J_PI}" />
+    <!--<xacro:property name="joint_3_lower_limit" value="${-4*J_PI}" />
+    <xacro:property name="joint_3_upper_limit" value="${4*J_PI}" />-->
     <xacro:property name="joint_3_velocity_limit" value="${36*J_PI/180}" />
     <xacro:property name="joint_3_torque_limit" value="40" />

Commit message: a

File: kinova-ros/kinova_description/urdf/j2n6s300.xacro (robot description, xacro)
@@ -59,6 +59,4 @@
     <xacro:property name="joint_2_lower_limit" value="${47/180*J_PI}" />
     <xacro:property name="joint_2_upper_limit" value="${313/180*J_PI}" />
-    <!--<xacro:property name="joint_2_lower_limit" value="${-4*J_PI}" />
-    <xacro:property name="joint_2_upper_limit" value="${4*J_PI}" />-->
     <xacro:property name="joint_2_velocity_limit" value="${36*J_PI/180}" />
     <xacro:property name="joint_2_torque_limit" value="80" />
@@ -70,6 +68,4 @@
     <xacro:property name="joint_3_lower_limit" value="${19/180*J_PI}" />
     <xacro:property name="joint_3_upper_limit" value="${341/180*J_PI}" />
-    <!--<xacro:property name="joint_3_lower_limit" value="${-4*J_PI}" />
-    <xacro:property name="joint_3_upper_limit" value="${4*J_PI}" />-->
     <xacro:property name="joint_3_velocity_limit" value="${36*J_PI/180}" />
     <xacro:property name="joint_3_torque_limit" value="40" />
